File: esp32/ESP32_SCM.kicad_sch (KiCad schematic)
At the start: 16 parts, among them J1 Head_Pan, J2 Head_Tilt, J3 Left_Arm, J4 Head_Pan, J5 INMP441, J6 MAX98357A, J7 HC_SR04, J8 PIR, J9 Touch, U1 ESP32-CAM (AI-Thinker)

Commit message: docs and esp32 schematic design change
Parts:
- added J10: FTDI, Connector_PinHeader_2.54mm:PinHeader_1x06_P2.54mm_Vertical, symbol Connector_Generic:Conn_01x06
- added R5: 10kohm, Resistor_SMD:R_0402_1005Metric, symbol Device:R
- C1: footprint (none) -> Capacitor_SMD:C_1210_3225Metric
- J1, J2, J3, J8, J9: footprint (none) -> Connector_PinHeader_2.54mm:PinHeader_1x03_P2.54mm_Vertical
- J4: value Head_Pan -> Right_Arm; footprint (none) -> Connector_PinHeader_2.54mm:PinHeader_1x03_P2.54mm_Vertical
- J5: footprint (none) -> Connector_PinHeader_2.54mm:PinHeader_1x06_P2.54mm_Vertical
- J6: footprint (none) -> Connector_PinHeader_2.54mm:PinHeader_1x05_P2.54mm_Vertical
- J7: footprint (none) -> Connector_PinHeader_2.54mm:PinHeader_1x04_P2.54mm_Vertical
- R1, R2, R3, R4: footprint (none) -> Resistor_SMD:R_0402_1005Metric
- U1: value ESP32-CAM (AI-Thinker) -> ESP32-WROOM-32
Connections:
- net +3V3: now also R5.1
- net +5V: now also J10.5V (Pin_1)
- net GND: now also J10.GND (Pin_2)
- net at U1.25 (IO0): now also J10.BOOT (Pin_5), R5.2
- net at R4.2, U1.3 (EN): now also J10.EN/RST (Pin_6)
- net at U1.34 (RXD0/IO3): now also J10.RX (Pin_4)
- net at U1.35 (TXD0/IO1): now also J10.TX (Pin_3)
- no-connect marks 18 -> 15
